Commit message: z coord problem in gazebo

File: urdf/amr.urdf (robot description, URDF)
Before this commit: robot amr, 4 links, 3 joints
Links:
- link base_link: geometry collision box ; visual mesh filename=package://amr/meshes/base_link.STL
- link left_wheel: geometry collision cylinder ; visual mesh filename=package://amr/meshes/left_wheel.STL
- link right_wheel: geometry collision cylinder ; visual mesh filename=package://amr/meshes/right_wheel.STL

Commit message: работает алгос, лагает газебо

File: urdf/amr.urdf (robot description, URDF)
Before this commit: robot amr, 4 links, 3 joints
Links:
- link base_link: geometry collision mesh filename=file:///workspace/src/dikom/meshes/base_link.STL; visual mesh filename=file:///workspace/src/dikom/meshes/base_link.STL
- link left_wheel: geometry collision mesh filename=file:///workspace/src/dikom/meshes/left_wheel.STL; visual mesh filename=file:///workspace/src/dikom/meshes/left_wheel.STL
- link lidar: geometry collision mesh filename=file:///workspace/src/dikom/meshes/lidar.STL; visual mesh filename=file:///workspace/src/dikom/meshes/lidar.STL
- link right_wheel: geometry collision mesh filename=file:///workspace/src/dikom/meshes/right_wheel.STL; visual mesh filename=file:///workspace/src/dikom/meshes/right_wheel.STL
